Commit message: modified shunk_egp50 xacro with stl files and transforms

File: workcell_description/urdf/shunk_egp50.xacro (robot description, xacro)
@@ -2,12 +2,12 @@
 <robot xmlns:xacro="http://www.ros.org/wiki/xacro" name="schunk_egp50">
     <xacro:macro name="schunk_egp50">
-    <!--GRIPPER-->
-    <!-- Base plate has 75mm diameter, 15mm thickness. Gripper body has 115mm height + pincers have 15mm height-->
         <xacro:property name="base_diamter" value="0.075" />
         <xacro:property name="base_length" value="0.015" />
         <xacro:property name="body_length" value="0.05" />
         <xacro:property name="body_width" value="0.03" />
-        <xacro:property name="body_height" value="0.115" />
-        <xacro:property name="pincer_height" value="0.015" />
+        <xacro:property name="body_height" value="0.0866" />
+        <xacro:property name="pincer_height" value="0.014" />
+        <xacro:property name="pincer_length" value="0.050" />
+        <xacro:property name="pincer_width" value="0.018" />
         <material name="blue">
             <color rgba="0 0 1 1" />
@@ -39,14 +39,12 @@
             <visual>
                 <geometry>
-                    <!--mesh filename="$(find ur_manipulation)/meshes/EGP50.stl" /-->
-                    <box size="${body_length} ${body_width} ${body_height}" />
+                    <mesh filename="package://workcell_description/meshes/Gripper.stl" scale="0.001 0.001 0.001"/>
                 </geometry>
+                <origin rpy="${pi/2} 0 0" xyz="${-body_length/2} ${body_width/2} ${-body_height/2}" />
                 <material name="green" />
-                <origin rpy="0 0 0" xyz="0 0 0" />
             </visual>
             <collision>
                 <geometry>
-                    <!--mesh filename="$(find ur_manipulation)/meshes/EGP50.stl" /-->
-                    <box size="${body_length} ${body_width} ${body_height}" />
+                    <mesh filename="package://workcell_description/meshes/Gripper.stl" scale="0.001 0.001 0.001"/>
                 </geometry>
                 <origin rpy="0 0 0" xyz="0 0 0" />
@@ -57,18 +55,38 @@
             </inertial>
         </link>
-        <!--Pincer block-->
-        <link name="egp50_pincer_link">
+        <!--Pincer block 1-->
+        <link name="egp50_pincer_1_link">
             <visual>
                 <geometry>
-                    <box size="${body_length} ${body_width} ${pincer_height}" />
+                    <mesh filename="package://workcell_description/meshes/Pincer_1.stl" scale="0.001 0.001 0.001"/>
                 </geometry>
-                <origin rpy="0 0 0" xyz="0 0 0" />
+                <origin rpy="${pi/2} 0 0" xyz="${-body_length/2} ${pincer_width/2} ${-body_height-pincer_height/2}" />
                 <material name="white" />
             </visual>
             <collision>
                 <geometry>
-                    <box size="${body_length} ${body_width} ${pincer_height}" />
+                    <mesh filename="package://workcell_description/meshes/Pincer_1.stl" scale="0.001 0.001 0.001"/>
                 </geometry>
-                <origin rpy="0 0 0" xyz="0 0 0" />
+                <origin rpy="${pi/2} 0 0" xyz="${-body_length/2} ${pincer_width/2} ${-body_height-pincer_height/2}" />
+            </collision>
+            <inertial>
+                <mass value="0.51" />
+                <inertia ixx="0.0007" iyy="0.0001" izz="0.0006" ixy="0.0" ixz="0.0" iyz="0.0" />
+            </inertial>
+        </link>
+        <!--Pincer block 2-->
+        <link name="egp50_pincer_2_link">
+            <visual>
+                <geometry>
+                    <mesh filename="package://workcell_description/meshes/Pincer_2.stl" scale="0.001 0.001 0.001"/>
+                </geometry>
+                <origin rpy="${pi/2} 0 0" xyz="${-body_length/2} ${pincer_width/2} ${-body_height-pincer_height/2}" />
+                <material name="blue" />
+            </visual>
+            <collision>
+                <geometry>
+                    <mesh filename="package://workcell_description/meshes/Pincer_2.stl" scale="0.001 0.001 0.001"/>
+                </geometry>
+                <origin rpy="${pi/2} 0 0" xyz="${-body_length/2} ${pincer_width/2} ${-body_height-pincer_height/2}" />
             </collision>
             <inertial>
@@ -85,11 +103,24 @@
             <origin xyz="0.0 0.0 ${base_length+body_height/2}" rpy="0.0 0.0 0.0" />
         </joint>
-        <joint name="egp50_pincer_joint" type="fixed">
+        <joint name="egp50_pincer_1_joint" type="prismatic">
             <parent link="egp50_body_link" />
-            <child link="egp50_pincer_link" />
+            <child link="egp50_pincer_1_link" />
             <origin xyz="0.0 0.0 ${body_height/2+pincer_height/2}" rpy="0.0 0.0 0.0" />
+            <!-- the motion of the pincer is along the X axis -->
+            <axis xyz="1 0 0"/>
+            <!-- the motion of the pincer is limited to the half of the gripper body length -->
+            <limit lower="0" upper="${body_length/2}" velocity="100" effort="100"/>
+        </joint>
+        <joint name="egp50_pincer_2_joint" type="prismatic">
+            <parent link="egp50_body_link" />
+            <child link="egp50_pincer_2_link" />
+            <origin xyz="0.0 0.002 ${body_height/2+pincer_height/2}" rpy="0.0 0.0 0.0" />
+            <!-- the motion of the pincer is along the X axis -->
+            <axis xyz="1 0 0"/>
+            <!-- the motion of the pincer is limited to the half of the gripper body length -->
+            <limit lower="0" upper="${body_length/2}" velocity="100" effort="100"/>
         </joint>
         <joint name="egp50_tip_joint" type="fixed">
-            <parent link="egp50_pincer_link" />
+            <parent link="egp50_pincer_1_link" />
             <child link="egp_50_tip" />
             <origin xyz="0.0 0.0 ${pincer_height/2}" rpy="0.0 0.0 0.0" />
