Commit message: added a grippy gripper urdf, modified shunk egp50 urdf and adding dependencies  ur_description&realsense2_description

File: workcell_description/urdf/gripper.xacro (robot description, xacro)
@@ -1,10 +1,16 @@
 <?xml version="1.0"?>
 <robot xmlns:xacro="http://www.ros.org/wiki/xacro" >
+    <!-- Choose which gripper to use -->
+    <xacro:property name="gripper_name" value="grippy" /> <!-- shunk_egp50 or grippy -->
     <joint name="robot_to_gripper_joint" type="fixed">
         <parent link="wrist_3_link" />
-        <child link="egp50_base_link" />
+        <child link="${gripper_name}_base_link" />
         <origin xyz="0.0 0.0 0.0" rpy="0.0 0.0 0.0" />
     </joint>
-    <xacro:include filename="$(find workcell_description)/urdf/shunk_egp50.xacro" />
-    <xacro:schunk_egp50 />
+    <!-- Uncomment 2 lines below and comment grippy to use shunk_egp50 Gripper  -->
+<!--     <xacro:include filename="$(find workcell_description)/urdf/shunk_egp50.xacro" />
+    <xacro:schunk_egp50 /> -->
+    <!-- Uncomment 2 lines below and comment shunk_egp50 to use grippy Gripper -->
+    <xacro:include filename="$(find workcell_description)/urdf/grippy.xacro" />
+    <xacro:grippy />
 </robot>

File: workcell_description/urdf/grippy.xacro (robot description, xacro)
@@ -1,13 +1,14 @@
 <?xml version="1.0"?>
-<robot xmlns:xacro="http://www.ros.org/wiki/xacro" name="schunk_egp50">
-    <xacro:macro name="schunk_egp50">
+<robot xmlns:xacro="http://www.ros.org/wiki/xacro" name="grippy">
+    <!-- This is GRIPPY, A gripper with exact measurements of Shunk EGP50 and with simlilar links and joints
+            This gripper is made with geometric shapes and can be extended as per your imagination.  -->
+    <xacro:macro name="grippy">
         <xacro:property name="base_diamter" value="0.075" />
         <xacro:property name="base_length" value="0.015" />
         <xacro:property name="body_length" value="0.05" />
         <xacro:property name="body_width" value="0.03" />
-        <xacro:property name="body_height" value="0.0866" />
-        <xacro:property name="body_height_max" value="0.01044" />
+        <xacro:property name="body_height" value="0.1044" />
         <xacro:property name="pincer_height" value="0.014" />
-        <xacro:property name="pincer_length" value="0.050" />
+        <xacro:property name="pincer_length" value="0.008" />
         <xacro:property name="pincer_width" value="0.018" />
         <material name="blue">
@@ -21,5 +22,5 @@
         </material>
         <!--Base plate-->
-        <link name="shunk_egp50_base_link">
+        <link name="grippy_base_link">
             <visual>
                 <geometry>
@@ -33,19 +34,39 @@
                     <cylinder length="${base_length}" radius="${base_diamter/2}" />
                 </geometry>
-                <origin rpy="0 0 0" xyz="0 0 0" />
+                <origin rpy="0 0 0" xyz="0 0 ${base_length/2}" />
             </collision>
         </link>
         <!--Main gripper-->
-        <link name="shunk_egp50_body_link">
+        <link name="grippy_body_link">
             <visual>
                 <geometry>
-                    <mesh filename="package://workcell_description/meshes/Gripper.stl" scale="0.001 0.001 0.001"/>
+                    <box size="${body_length} ${body_width} ${body_height}" />
                 </geometry>
-                <origin rpy="${pi/2} 0 0" xyz="${-body_length/2} ${body_width/2} ${-body_height/2}" />
                 <material name="green" />
+                <origin rpy="0 0 0 " xyz="0 0 ${body_height/2}" />
             </visual>
             <collision>
                 <geometry>
-                    <mesh filename="package://workcell_description/meshes/Gripper.stl" scale="0.001 0.001 0.001"/>
+                    <box size="${body_length} ${body_width} ${body_height}" />
+                </geometry>
+                <origin rpy="0 0 0 " xyz="0 0 ${body_height/2}" />
+            </collision>
+            <inertial>
+                <mass value="0.51" />
+                <inertia ixx="0.0007" iyy="0.0001" izz="0.0006" ixy="0.0" ixz="0.0" iyz="0.0" />
+            </inertial>
+        </link>
+        <!--Pincer block 1-->
+        <link name="grippy_left_pincer_link">
+            <visual>
+                <geometry>
+                    <box size="${pincer_length} ${pincer_width} ${pincer_height}" />
+                </geometry>
+                <origin rpy="0 0 0" xyz="0 0 0" />
+                <material name="white" />
+            </visual>
+            <collision>
+                <geometry>
+                    <box size="${pincer_length} ${pincer_width} ${pincer_height}" />
                 </geometry>
                 <origin rpy="0 0 0" xyz="0 0 0" />
@@ -56,38 +77,18 @@
             </inertial>
         </link>
-        <!--Pincer block 1-->
-        <link name="shunk_egp50_pincer_1_link">
+        <!--Pincer block 2-->
+        <link name="grippy_right_pincer_link">
             <visual>
                 <geometry>
-                    <mesh filename="package://workcell_description/meshes/Pincer_1.stl" scale="0.001 0.001 0.001"/>
+                    <box size="${pincer_length} ${pincer_width} ${pincer_height}" />
                 </geometry>
-                <origin rpy="${pi/2} 0 0" xyz="${-body_length/2} ${pincer_width/2} ${-body_height-pincer_height/2}" />
+                <origin rpy="0 0 0" xyz="0 0 0" />
                 <material name="white" />
             </visual>
             <collision>
                 <geometry>
-                    <mesh filename="package://workcell_description/meshes/Pincer_1.stl" scale="0.001 0.001 0.001"/>
+                    <box size="${pincer_length} ${pincer_width} ${pincer_height}" />
                 </geometry>
-                <origin rpy="${pi/2} 0 0" xyz="${-body_length/2} ${pincer_width/2} ${-body_height-pincer_height/2}" />
-            </collision>
-            <inertial>
-                <mass value="0.51" />
-                <inertia ixx="0.0007" iyy="0.0001" izz="0.0006" ixy="0.0" ixz="0.0" iyz="0.0" />
-            </inertial>
-        </link>
-        <!--Pincer block 2-->
-        <link name="shunk_egp50_pincer_2_link">
-            <visual>
-                <geometry>
-                    <mesh filename="package://workcell_description/meshes/Pincer_2.stl" scale="0.001 0.001 0.001"/>
-                </geometry>
-                <origin rpy="${pi/2} 0 0" xyz="${-body_length/2} ${pincer_width/2} ${-body_height-pincer_height/2}" />
-                <material name="blue" />
-            </visual>
-            <collision>
-                <geometry>
-                    <mesh filename="package://workcell_description/meshes/Pincer_2.stl" scale="0.001 0.001 0.001"/>
-                </geometry>
-                <origin rpy="${pi/2} 0 0" xyz="${-body_length/2} ${pincer_width/2} ${-body_height-pincer_height/2}" />
+                <origin rpy="0 0 0" xyz="0 0 0" />
             </collision>
             <inertial>
@@ -99,31 +100,31 @@
         <link name="tool_tip" />
         <!-- Joints-->
-        <joint name="shunk_egp50_body_joint" type="fixed">
-            <parent link="shunk_egp50_base_link" />
-            <child link="shunk_egp50_body_link" />
-            <origin xyz="0.0 0.0 ${base_length+body_height/2}" rpy="0.0 0.0 0.0" />
+        <joint name="grippy_body_joint" type="fixed">
+            <parent link="grippy_base_link" />
+            <child link="grippy_body_link" />
+            <origin xyz="0.0 0.0 ${base_length}" rpy="0.0 0.0 0.0" />
         </joint>
-        <joint name="shunk_egp50_pincer_1_joint" type="prismatic">
-            <parent link="shunk_egp50_body_link" />
-            <child link="shunk_egp50_pincer_1_link" />
-            <origin xyz="0.0 0.0 ${body_height/2+pincer_height/2}" rpy="0.0 0.0 0.0" />
+        <joint name="grippy_pincer_left_joint" type="prismatic">
+            <parent link="grippy_body_link" />
+            <child link="grippy_left_pincer_link" />
+            <origin xyz="${-body_length/2+pincer_length/2} 0 ${body_height+pincer_height/2}" rpy="0 0 0" />
             <!-- the motion of the pincer is along the X axis -->
-            <axis xyz="1 0 0"/>
+            <axis xyz="1 0 0" />
             <!-- the motion of the pincer is limited to the half of the gripper body length -->
-            <limit lower="${-body_length/16}" upper="${body_length/16}" velocity="100" effort="100"/>
+            <limit lower="0" upper="${body_length/4}" velocity="100" effort="100" />
         </joint>
-        <joint name="shunk_egp50_pincer_2_joint" type="prismatic">
-            <parent link="shunk_egp50_body_link" />
-            <child link="shunk_egp50_pincer_2_link" />
-            <origin xyz="0.0 0.002 ${body_height/2+pincer_height/2}" rpy="0.0 0.0 0.0" />
+        <joint name="grippy_pincer_right_joint" type="prismatic">
+            <parent link="grippy_body_link" />
+            <child link="grippy_right_pincer_link" />
+            <origin xyz="${body_length/2-pincer_length/2} 0 ${body_height+pincer_height/2}" rpy="0.0 0.0 0.0" />
             <!-- the motion of the pincer is along the X axis -->
-            <axis xyz="1 0 0"/>
+            <axis xyz="-1 0 0" />
             <!-- the motion of the pincer is limited to the half of the gripper body length -->
-            <limit lower="${body_length/16}" upper="${-body_length/16}" velocity="100" effort="100"/>
+            <limit lower="0" upper="${body_length/4}" velocity="100" effort="100" />
         </joint>
-        <joint name="shunk_egp50_tip_joint" type="fixed">
-            <parent link="shunk_egp50_base_link" />
+        <joint name="grippy_tip_joint" type="fixed">
+            <parent link="grippy_body_link" />
             <child link="tool_tip" />
-            <origin xyz="0 0 ${body_height_max}" rpy="0.0 0.0 0.0" />
+            <origin xyz="0.0 0.0 ${body_height}" rpy="0.0 0.0 0.0" />
         </joint>
     </xacro:macro>

File: workcell_description/urdf/robotcell.xacro (robot description, xacro)
@@ -3,15 +3,7 @@
     <link name="world">
     </link>
-    <xacro:property name="robotcell_length" value="1" />
-    <xacro:property name="robotcell_width" value="0.5" />
-    <xacro:property name="robotcell_height" value="1" />
-    <joint name="world_to_robotcell_joint" type="fixed">
-        <parent link="world" />
-        <child link="robotcell_link" />
-        <origin xyz="0 0 0" rpy="0 0 0" />
-    </joint>
-    <link name="robotcell_link">
+<!--     <link name="shield_front">
         <visual>
-            <origin rpy="0 ${-pi} ${-pi/2}" xyz="-0.5 -0.5 2" />
+            <origin rpy="0 0 0" xyz="0 0 0" />
             <geometry>
                 <mesh filename="package://workcell_description/meshes/Robotcell.stl" scale="0.001 0.001 0.001"/>
@@ -25,3 +17,34 @@
         </collision>
     </link>
+    <link name="shield_rear">
+    </link>
+    <link name="shield_left">
+    </link>
+    <link name="shield_right">
+    </link> -->
+    <xacro:property name="robot_base_length" value="0.5" />
+    <xacro:property name="robot_base_width" value="0.5" />
+    <xacro:property name="robot_base_height" value="2" />
+    <xacro:property name="robotcell_length" value="1" />
+    <xacro:property name="robotcell_width" value="1" />
+    <xacro:property name="robotcell_height" value="4" />
+    <joint name="world_to_robotcell_joint" type="fixed">
+        <parent link="world" />
+        <child link="robotcell_link" />
+        <origin xyz="0 0 0" rpy="0 0 0" />
+    </joint>
+    <link name="robotcell_link">
+        <visual>
+            <origin rpy="0 ${-pi} ${-pi/2}" xyz="${-robot_base_length} ${-robot_base_width} ${robot_base_height}" />
+            <geometry>
+                <mesh filename="package://workcell_description/meshes/Robotcell.stl" scale="0.001 0.001 0.001"/>
+            </geometry>
+        </visual>
+        <collision>
+            <origin rpy="0 ${-pi} ${-pi/2}" xyz="${-robot_base_length} ${-robot_base_width} ${robot_base_height}" />
+            <geometry>
+                <mesh filename="package://workcell_description/meshes/Robotcell.stl" scale="0.001 0.001 0.001" />
+            </geometry>
+        </collision>
+    </link>
 </robot>
