Commit message: added launch files and modified parameters in the urdf files

File: workcell_description/urdf/camera.xacro (robot description, xacro)
@@ -1,6 +1,6 @@
 <?xml version="1.0"?>
 <robot xmlns:xacro="http://www.ros.org/wiki/xacro" >
-    <xacro:property name="robotcell_length" value="1" />
-    <xacro:property name="robotcell_width" value="0.5" />
+    <xacro:property name="robotcell_length" value="0.5" />
+    <xacro:property name="robotcell_width" value="-0.5" />
     <xacro:property name="robotcell_height" value="1" />
     <xacro:include filename="$(find realsense2_description)/urdf/_d435.urdf.xacro" />
@@ -13,5 +13,5 @@
         add_plug="$(arg add_plug)"
         use_mesh="$(arg use_mesh)">
-        <origin xyz="-${robotcell_length/2} -${robotcell_width} -${robotcell_height}" rpy="0 -${pi/2} 0" />
+        <origin xyz="${robotcell_length} ${robotcell_width} ${robotcell_height}" rpy="${pi/2} ${pi/2} ${-pi}" />
     </xacro:sensor_d435>
 </robot>

File: workcell_description/urdf/robotcell.xacro (robot description, xacro)
@@ -1,5 +1,6 @@
 <?xml version="1.0"?>
 <robot xmlns:xacro="http://www.ros.org/wiki/xacro" >
-    <link name="world" />
+    <link name="world">
+    </link>
     <xacro:property name="robotcell_length" value="1" />
     <xacro:property name="robotcell_width" value="0.5" />
@@ -8,17 +9,17 @@
         <parent link="world" />
         <child link="robotcell_link" />
-        <origin xyz="-${robotcell_length/2} -${robotcell_width/2} 0" rpy="0 0 0" />
+        <origin xyz="0 0 0" rpy="0 0 0" />
     </joint>
     <link name="robotcell_link">
         <visual>
-            <origin rpy="0.0 0 0" xyz="0 0 0" />
+            <origin rpy="0 ${-pi} ${-pi/2}" xyz="-0.5 -0.5 2" />
             <geometry>
-                <mesh filename="package://workcell_description/meshes/Robotcell.stl" />
+                <mesh filename="package://workcell_description/meshes/Robotcell.stl" scale="0.001 0.001 0.001"/>
             </geometry>
         </visual>
         <collision>
-            <origin rpy="0.0 0 0" xyz="0 0 0" />
+            <origin rpy="0 0 0 " xyz="0 0 0" />
             <geometry>
-                <mesh filename="package://workcell_description/meshes/Robotcell.stl" />
+                <mesh filename="package://workcell_description/meshes/Robotcell.stl" scale="0.001 0.001 0.001" />
             </geometry>
         </collision>

Commit message: modified urdf xacros for the workcell

File: workcell_description/urdf/camera.xacro (robot description, xacro)
@@ -1,7 +1,13 @@
 <?xml version="1.0"?>
 <robot xmlns:xacro="http://www.ros.org/wiki/xacro" >
-    <xacro:property name="robotcell_length" value="0.5" />
-    <xacro:property name="robotcell_width" value="-0.5" />
-    <xacro:property name="robotcell_height" value="1" />
+    <xacro:property name="robot_base_length" value="0.30" />
+    <xacro:property name="robot_base_width" value="0.52" />
+    <xacro:property name="robot_base_offset_length" value="0.45" />
+    <xacro:property name="robot_base_offset_width" value="0.02" />
+    <xacro:property name="robot_base_height" value="0.99" />
+    <xacro:property name="robotcell_length" value="1.44" />
+    <xacro:property name="robotcell_width" value="0.94" />
+    <xacro:property name="robotcell_height" value="1.16" />
+    <xacro:property name="shield_thickness" value="0.03" />
     <xacro:include filename="$(find realsense2_description)/urdf/_d435.urdf.xacro" />
     <xacro:arg name="use_nominal_extrinsics" default="false"/>
@@ -13,5 +19,7 @@
         add_plug="$(arg add_plug)"
         use_mesh="$(arg use_mesh)">
-        <origin xyz="${robotcell_length} ${robotcell_width} ${robotcell_height}" rpy="${pi/2} ${pi/2} ${-pi}" />
+        <origin xyz="0  0  ${robotcell_height+robot_base_height-shield_thickness}" rpy="${pi/2} ${pi/2} 0" />
     </xacro:sensor_d435>
 </robot>
+<!-- ${robotcell_length/2} ${robotcell_width/2}
+${pi/2} ${pi/2} -->

File: workcell_description/urdf/gripper.xacro (robot description, xacro)
@@ -2,5 +2,5 @@
 <robot xmlns:xacro="http://www.ros.org/wiki/xacro" >
     <!-- Choose which gripper to use -->
-    <xacro:property name="gripper_name" value="grippy" /> <!-- shunk_egp50 or grippy -->
+    <xacro:property name="gripper_name" value="shunk_clone" /> <!-- shunk_egp50 or shunk_clone -->
     <joint name="robot_to_gripper_joint" type="fixed">
         <parent link="wrist_3_link" />
@@ -8,9 +8,9 @@
         <origin xyz="0.0 0.0 0.0" rpy="0.0 0.0 0.0" />
     </joint>
-    <!-- Uncomment 2 lines below and comment grippy to use shunk_egp50 Gripper  -->
+    <!-- Uncomment 2 lines below and comment shunk_clone to use shunk_egp50 Gripper  -->
 <!--     <xacro:include filename="$(find workcell_description)/urdf/shunk_egp50.xacro" />
     <xacro:schunk_egp50 /> -->
-    <!-- Uncomment 2 lines below and comment shunk_egp50 to use grippy Gripper -->
-    <xacro:include filename="$(find workcell_description)/urdf/grippy.xacro" />
-    <xacro:grippy />
+    <!-- Uncomment 2 lines below and comment shunk_egp50 to use shunk_clone Gripper -->
+    <xacro:include filename="$(find workcell_description)/urdf/shunk_clone.xacro" />
+    <xacro:shunk_clone />
 </robot>

File: workcell_description/urdf/robot.xacro (robot description, xacro)
@@ -1,11 +1,17 @@
 <?xml version="1.0"?>
 <robot xmlns:xacro="http://www.ros.org/wiki/xacro">
-    <xacro:property name="robotcell_length" value="1" />
-    <xacro:property name="robotcell_width" value="0.5" />
-    <xacro:property name="robotcell_height" value="1" />
+    <xacro:property name="robot_base_length" value="0.30" />
+    <xacro:property name="robot_base_width" value="0.52" />
+    <xacro:property name="robot_base_offset_length" value="0.45" />
+    <xacro:property name="robot_base_offset_width" value="0.02" />
+    <xacro:property name="robot_base_height" value="0.99" />
+    <xacro:property name="robotcell_length" value="1.44" />
+    <xacro:property name="robotcell_width" value="0.94" />
+    <xacro:property name="robotcell_height" value="1.16" />
+    <xacro:property name="shield_thickness" value="0.03" />
     <joint name="robotcell_to_robot_joint" type="fixed">
         <parent link="robotcell_link" />
         <child link="base_link" />
-        <origin xyz="0 0 0" rpy="0 0 0" />
+        <origin xyz="${robot_base_offset_length} ${-robot_base_offset_width} ${robot_base_height}" rpy="0 0 ${-pi}" />
     </joint>
     <!-- robot name parameter -->

File: workcell_description/urdf/robotcell.xacro (robot description, xacro)
@@ -3,30 +3,10 @@
     <link name="world">
     </link>
-<!--     <link name="shield_front">
-        <visual>
-            <origin rpy="0 0 0" xyz="0 0 0" />
-            <geometry>
-                <mesh filename="package://workcell_description/meshes/Robotcell.stl" scale="0.001 0.001 0.001"/>
-            </geometry>
-        </visual>
-        <collision>
-            <origin rpy="0 0 0 " xyz="0 0 0" />
-            <geometry>
-                <mesh filename="package://workcell_description/meshes/Robotcell.stl" scale="0.001 0.001 0.001" />
-            </geometry>
-        </collision>
-    </link>
-    <link name="shield_rear">
-    </link>
-    <link name="shield_left">
-    </link>
-    <link name="shield_right">
-    </link> -->
-    <xacro:property name="robot_base_length" value="0.5" />
-    <xacro:property name="robot_base_width" value="0.5" />
-    <xacro:property name="robot_base_height" value="2" />
-    <xacro:property name="robotcell_length" value="1" />
-    <xacro:property name="robotcell_width" value="1" />
-    <xacro:property name="robotcell_height" value="4" />
+    <xacro:property name="robot_base_length" value="0.30" />
+    <xacro:property name="robot_base_width" value="0.52" />
+    <xacro:property name="robot_base_height" value="0.99" />
+    <xacro:property name="robotcell_length" value="1.44" />
+    <xacro:property name="robotcell_width" value="0.94" />
+    <xacro:property name="robotcell_height" value="1.13" />
     <joint name="world_to_robotcell_joint" type="fixed">
         <parent link="world" />

File: workcell_description/urdf/shunk_clone.xacro (robot description, xacro)
@@ -1,7 +1,7 @@
 <?xml version="1.0"?>
-<robot xmlns:xacro="http://www.ros.org/wiki/xacro" name="grippy">
+<robot xmlns:xacro="http://www.ros.org/wiki/xacro" name="shunk_clone">
     <!-- This is GRIPPY, A gripper with exact measurements of Shunk EGP50 and with simlilar links and joints
             This gripper is made with geometric shapes and can be extended as per your imagination.  -->
-    <xacro:macro name="grippy">
+    <xacro:macro name="shunk_clone">
         <xacro:include filename="inertial_macros.xacro"/>
         <xacro:property name="base_diameter" value="0.075" />
@@ -14,8 +14,8 @@
         <xacro:property name="pincer_width" value="0.018" />
         <material name="blue">
-            <color rgba="0 0 1 1" />
+            <color rgba="0 0.2 1 1" />
         </material>
         <material name="green">
-            <color rgba="0 1 0 1" />
+            <color rgba="0 0.9 0.3 1" />
         </material>
         <material name="white">
@@ -23,5 +23,5 @@
         </material>
         <!--Base plate-->
-        <link name="grippy_base_link">
+        <link name="shunk_clone_base_link">
             <visual>
                 <geometry>
@@ -42,5 +42,5 @@
         </link>
         <!--Main gripper-->
-        <link name="grippy_body_link">
+        <link name="shunk_clone_body_link">
             <visual>
                 <geometry>
@@ -56,14 +56,10 @@
                 <origin rpy="0 0 0 " xyz="0 0 ${body_height/2}" />
             </collision>
-            <inertial>
-                <mass value="0.51" />
-                <inertia ixx="0.0007" iyy="0.0001" izz="0.0006" ixy="0.0" ixz="0.0" iyz="0.0" />
-            </inertial>
-            <xacro:inertial_box mass="0.5" x="${body_length}" y="${body_width}" z="${body_height}">
+            <xacro:inertial_box mass="0.51" x="${body_length}" y="${body_width}" z="${body_height}">
                 <origin rpy="0 0 0 " xyz="0 0 ${body_height/2}" />
             </xacro:inertial_box>
         </link>
         <!--Pincer block 1-->
-        <link name="grippy_left_pincer_link">
+        <link name="shunk_clone_left_pincer_link">
             <visual>
                 <geometry>
@@ -84,5 +80,5 @@
         </link>
         <!--Pincer block 2-->
-        <link name="grippy_right_pincer_link">
+        <link name="shunk_clone_right_pincer_link">
             <visual>
                 <geometry>
@@ -105,12 +101,12 @@
         <link name="tool_tip" />
         <!-- Joints-->
-        <joint name="grippy_body_joint" type="fixed">
-            <parent link="grippy_base_link" />
-            <child link="grippy_body_link" />
+        <joint name="shunk_clone_body_joint" type="fixed">
+            <parent link="shunk_clone_base_link" />
+            <child link="shunk_clone_body_link" />
             <origin xyz="0.0 0.0 ${base_length}" rpy="0.0 0.0 0.0" />
         </joint>
-        <joint name="grippy_pincer_left_joint" type="prismatic">
-            <parent link="grippy_body_link" />
-            <child link="grippy_left_pincer_link" />
+        <joint name="shunk_clone_pincer_left_joint" type="prismatic">
+            <parent link="shunk_clone_body_link" />
+            <child link="shunk_clone_left_pincer_link" />
             <origin xyz="${-body_length/2+pincer_length/2} 0 ${body_height+pincer_height/2}" rpy="0 0 0" />
             <!-- the motion of the pincer is along the X axis -->
@@ -119,7 +115,7 @@
             <limit lower="0" upper="${body_length/4}" velocity="100" effort="100" />
         </joint>
-        <joint name="grippy_pincer_right_joint" type="prismatic">
-            <parent link="grippy_body_link" />
-            <child link="grippy_right_pincer_link" />
+        <joint name="shunk_clone_pincer_right_joint" type="prismatic">
+            <parent link="shunk_clone_body_link" />
+            <child link="shunk_clone_right_pincer_link" />
             <origin xyz="${body_length/2-pincer_length/2} 0 ${body_height+pincer_height/2}" rpy="0.0 0.0 0.0" />
             <!-- the motion of the pincer is along the X axis -->
@@ -128,6 +124,6 @@
             <limit lower="0" upper="${body_length/4}" velocity="100" effort="100" />
         </joint>
-        <joint name="grippy_tip_joint" type="fixed">
-            <parent link="grippy_body_link" />
+        <joint name="shunk_clone_tip_joint" type="fixed">
+            <parent link="shunk_clone_body_link" />
             <child link="tool_tip" />
             <origin xyz="0.0 0.0 ${body_height}" rpy="0.0 0.0 0.0" />

File: workcell_description/urdf/shunk_egp50.xacro (robot description, xacro)
@@ -13,8 +13,8 @@
         <xacro:property name="pincer_width" value="0.018" />
         <material name="blue">
-            <color rgba="0 0 1 1" />
+            <color rgba="0 0.2 1 1" />
         </material>
         <material name="green">
-            <color rgba="0 1 0 1" />
+            <color rgba="0 0.9 0.3 1" />
         </material>
         <material name="white">

File: workcell_description/urdf/workcell.urdf.xacro (robot description, xacro)
@@ -2,5 +2,5 @@
 <robot xmlns:xacro="http://www.ros.org/wiki/xacro" name="ur5e_workcell">
     <!-- loading robotcell from workcell_description package-->
-    <xacro:include filename="$(find workcell_description)/urdf/robotcell.xacro" />
+    <xacro:include filename="$(find workcell_description)/urdf/robot_cage.xacro" />
     <!-- loading robot  from workcell_description package-->
     <xacro:include filename="$(find workcell_description)/urdf/robot.xacro" />

Commit message: fixing launch files, gazebo issues and urdf

File: workcell_description/urdf/camera.xacro (robot description, xacro)
@@ -22,4 +22,2 @@
     </xacro:sensor_d435>
 </robot>
-<!-- ${robotcell_length/2} ${robotcell_width/2}
-${pi/2} ${pi/2} -->

File: workcell_description/urdf/gazebo_control.xacro (robot description, xacro)
@@ -1,16 +1,4 @@
 <?xml version="1.0"?>
 <robot xmlns:xacro="http://www.ros.org/wiki/xacro">
- <!--    <gazebo reference="shunk_egp50_base_link">
-        <material>Gazebo/Blue</material>
-    </gazebo>
-    <gazebo reference="shunk_egp50_body_link">
-        <material>Gazebo/Green</material>
-    </gazebo>
-    <gazebo reference="shunk_egp50_pincer_1_link">
-        <material>Gazebo/White</material>
-    </gazebo>
-    <gazebo reference="shunk_egp50_pincer_2_link">
-        <material>Gazebo/Blue</material>
-    </gazebo> -->
     <!-- This plugin will publish the joint_states for the selected joints
             (which robot_state_publisher can then use to broadcast the approprate tf). -->
@@ -18,5 +6,13 @@
         <plugin name="gazebo_ros_joint_state_publisher"
             filename="libgazebo_ros_joint_state_publisher.so">
-            <update_rate>20</update_rate>
+            <update_rate>200</update_rate>
+            <joint_name>shoulder_pan_joint</joint_name>
+            <joint_name>shoulder_lift_joint</joint_name>
+            <joint_name>elbow joint</joint_name>
+            <joint_name>wrist_1_joint</joint_name>
+            <joint_name>wrist_2_joint</joint_name>
+            <joint_name>wrist_3_joint</joint_name>
+            <joint_name>shunk_egp50_pincer_1_joint</joint_name>
+            <joint_name>shunk_egp50_pincer_2_joint</joint_name>
         </plugin>
     </gazebo>
@@ -26,9 +22,9 @@
         <plugin name="gazebo_ros_joint_pose_trajectory"
             filename="libgazebo_ros_joint_pose_trajectory.so">
-            <update_rate>20</update_rate>
+            <update_rate>200</update_rate>
         </plugin>
     </gazebo>
     <!-- This plugin is to include the depth camera -->
-<!--     <gazebo reference="camera_link">
+    <gazebo reference="camera_link">
         <material>Gazebo/Red</material>
         <sensor name="camera" type="depth">
@@ -49,4 +45,5 @@
             </camera>
             <plugin name="camera_controller" filename="libgazebo_ros_camera.so">
+                <camera_name>realsense_camera</camera_name>
                 <frame_name>camera_link_optical</frame_name>
                 <min_depth>0.1</min_depth>
@@ -54,4 +51,4 @@
             </plugin>
         </sensor>
-    </gazebo> -->
+    </gazebo>
 </robot>

File: workcell_description/urdf/gripper.xacro (robot description, xacro)
@@ -2,15 +2,15 @@
 <robot xmlns:xacro="http://www.ros.org/wiki/xacro" >
     <!-- Choose which gripper to use -->
-    <xacro:property name="gripper_name" value="shunk_clone" /> <!-- shunk_egp50 or shunk_clone -->
+    <xacro:property name="gripper_name" value="shunk_egp50" /> <!-- shunk_egp50 / shunk_clone -->
     <joint name="robot_to_gripper_joint" type="fixed">
-        <parent link="wrist_3_link" />
+        <parent link="tool0" />
         <child link="${gripper_name}_base_link" />
         <origin xyz="0.0 0.0 0.0" rpy="0.0 0.0 0.0" />
     </joint>
     <!-- Uncomment 2 lines below and comment shunk_clone to use shunk_egp50 Gripper  -->
-<!--     <xacro:include filename="$(find workcell_description)/urdf/shunk_egp50.xacro" />
-    <xacro:schunk_egp50 /> -->
+    <xacro:include filename="$(find workcell_description)/urdf/shunk_egp50.xacro" />
+    <xacro:schunk_egp50 />
     <!-- Uncomment 2 lines below and comment shunk_egp50 to use shunk_clone Gripper -->
-    <xacro:include filename="$(find workcell_description)/urdf/shunk_clone.xacro" />
-    <xacro:shunk_clone />
+<!--     <xacro:include filename="$(find workcell_description)/urdf/shunk_clone.xacro" />
+    <xacro:shunk_clone /> -->
 </robot>

File: workcell_description/urdf/robot.xacro (robot description, xacro)
@@ -51,6 +51,6 @@
     <xacro:arg name="use_fake_hardware" default="false" />
     <xacro:arg name="fake_sensor_commands" default="false" />
-    <xacro:arg name="sim_gazebo" default="false" />
-    <xacro:arg name="sim_ignition" default="false" />
+    <xacro:arg name="sim_gazebo" default="true" />
+    <xacro:arg name="sim_ignition" default="true" />
     <xacro:arg name="simulation_controllers" default="" />
     <!-- initial position for simulations (Fake Hardware, Gazebo, Ignition) -->

File: workcell_description/urdf/workcell.urdf.xacro (robot description, xacro)
@@ -2,5 +2,5 @@
 <robot xmlns:xacro="http://www.ros.org/wiki/xacro" name="ur5e_workcell">
     <!-- loading robotcell from workcell_description package-->
-    <xacro:include filename="$(find workcell_description)/urdf/robot_cage.xacro" />
+    <xacro:include filename="$(find workcell_description)/urdf/robot_cell_clone.xacro" />
     <!-- loading robot  from workcell_description package-->
     <xacro:include filename="$(find workcell_description)/urdf/robot.xacro" />
@@ -9,4 +9,5 @@
     <!-- loading camera from workcell_description package-->
     <xacro:include filename="$(find workcell_description)/urdf/camera.xacro" />
+    <!-- loading gazebo plugins-->
     <xacro:include filename="$(find workcell_description)/urdf/gazebo_control.xacro" />
 </robot>
