Commit message: updated intertial elements in urdf and added docker-gui docs

File: workcell_description/urdf/gazebo_control.xacro (robot description, xacro)
@@ -1,16 +1,16 @@
 <?xml version="1.0"?>
 <robot xmlns:xacro="http://www.ros.org/wiki/xacro">
-    <gazebo reference="egp50_base_link">
+ <!--    <gazebo reference="shunk_egp50_base_link">
         <material>Gazebo/Blue</material>
     </gazebo>
-    <gazebo reference="egp50_body_link">
+    <gazebo reference="shunk_egp50_body_link">
         <material>Gazebo/Green</material>
     </gazebo>
-    <gazebo reference="egp50_pincer_1_link">
+    <gazebo reference="shunk_egp50_pincer_1_link">
         <material>Gazebo/White</material>
     </gazebo>
-    <gazebo reference="egp50_pincer_2_link">
+    <gazebo reference="shunk_egp50_pincer_2_link">
         <material>Gazebo/Blue</material>
-    </gazebo>
+    </gazebo> -->
     <!-- This plugin will publish the joint_states for the selected joints
             (which robot_state_publisher can then use to broadcast the approprate tf). -->
@@ -30,5 +30,5 @@
     </gazebo>
     <!-- This plugin is to include the depth camera -->
-    <gazebo reference="camera_link">
+<!--     <gazebo reference="camera_link">
         <material>Gazebo/Red</material>
         <sensor name="camera" type="depth">
@@ -54,4 +54,4 @@
             </plugin>
         </sensor>
-    </gazebo>
+    </gazebo> -->
 </robot>

File: workcell_description/urdf/grippy.xacro (robot description, xacro)
@@ -4,5 +4,6 @@
             This gripper is made with geometric shapes and can be extended as per your imagination.  -->
     <xacro:macro name="grippy">
-        <xacro:property name="base_diamter" value="0.075" />
+        <xacro:include filename="inertial_macros.xacro"/>
+        <xacro:property name="base_diameter" value="0.075" />
         <xacro:property name="base_length" value="0.015" />
         <xacro:property name="body_length" value="0.05" />
@@ -25,5 +26,5 @@
             <visual>
                 <geometry>
-                    <cylinder length="${base_length}" radius="${base_diamter/2}" />
+                    <cylinder length="${base_length}" radius="${base_diameter/2}" />
                 </geometry>
                 <material name="blue" />
@@ -32,8 +33,11 @@
             <collision>
                 <geometry>
-                    <cylinder length="${base_length}" radius="${base_diamter/2}" />
+                    <cylinder length="${base_length}" radius="${base_diameter/2}" />
                 </geometry>
                 <origin rpy="0 0 0" xyz="0 0 ${base_length/2}" />
             </collision>
+            <xacro:inertial_cylinder mass="0.2" length="${base_length}" radius="${base_diameter/2}">
+                <origin rpy="0 0 0" xyz="0 0 ${base_length/2}" />
+            </xacro:inertial_cylinder>
         </link>
         <!--Main gripper-->
@@ -56,4 +60,7 @@
                 <inertia ixx="0.0007" iyy="0.0001" izz="0.0006" ixy="0.0" ixz="0.0" iyz="0.0" />
             </inertial>
+            <xacro:inertial_box mass="0.5" x="${body_length}" y="${body_width}" z="${body_height}">
+                <origin rpy="0 0 0 " xyz="0 0 ${body_height/2}" />
+            </xacro:inertial_box>
         </link>
         <!--Pincer block 1-->
@@ -72,8 +79,7 @@
                 <origin rpy="0 0 0" xyz="0 0 0" />
             </collision>
-            <inertial>
-                <mass value="0.51" />
-                <inertia ixx="0.0007" iyy="0.0001" izz="0.0006" ixy="0.0" ixz="0.0" iyz="0.0" />
-            </inertial>
+            <xacro:inertial_box mass="0.1" x="${pincer_length}" y="${pincer_width}" z="${pincer_height}">
+                <origin rpy="0 0 0" xyz="0 0 0" />
+            </xacro:inertial_box>
         </link>
         <!--Pincer block 2-->
@@ -92,8 +98,7 @@
                 <origin rpy="0 0 0" xyz="0 0 0" />
             </collision>
-            <inertial>
-                <mass value="0.51" />
-                <inertia ixx="0.0007" iyy="0.0001" izz="0.0006" ixy="0.0" ixz="0.0" iyz="0.0" />
-            </inertial>
+            <xacro:inertial_box mass="0.1" x="${pincer_length}" y="${pincer_width}" z="${pincer_height}">
+                <origin rpy="0 0 0" xyz="0 0 0" />
+            </xacro:inertial_box>
         </link>
         <!-- Virtual link for visualizytion and planning-->

File: workcell_description/urdf/shunk_egp50.xacro (robot description, xacro)
@@ -2,5 +2,6 @@
 <robot xmlns:xacro="http://www.ros.org/wiki/xacro" name="schunk_egp50">
     <xacro:macro name="schunk_egp50">
-        <xacro:property name="base_diamter" value="0.075" />
+        <xacro:include filename="inertial_macros.xacro" />
+        <xacro:property name="base_diameter" value="0.075" />
         <xacro:property name="base_length" value="0.015" />
         <xacro:property name="body_length" value="0.05" />
@@ -24,5 +25,5 @@
             <visual>
                 <geometry>
-                    <cylinder length="${base_length}" radius="${base_diamter/2}" />
+                    <cylinder length="${base_length}" radius="${base_diameter/2}" />
                 </geometry>
                 <material name="blue" />
@@ -31,8 +32,11 @@
             <collision>
                 <geometry>
-                    <cylinder length="${base_length}" radius="${base_diamter/2}" />
+                    <cylinder length="${base_length}" radius="${base_diameter/2}" />
                 </geometry>
-                <origin rpy="0 0 0" xyz="0 0 0" />
+                <origin rpy="0 0 0" xyz="0 0 ${base_length/2}" />
             </collision>
+            <xacro:inertial_cylinder mass="0.2" length="${base_length}" radius="${base_diameter/2}">
+                <origin rpy="0 0 0" xyz="0 0 ${base_length/2}" />
+            </xacro:inertial_cylinder>
         </link>
         <!--Main gripper-->
@@ -40,5 +44,5 @@
             <visual>
                 <geometry>
-                    <mesh filename="package://workcell_description/meshes/Gripper.stl" scale="0.001 0.001 0.001"/>
+                    <mesh filename="package://workcell_description/meshes/Gripper.stl" scale="0.001 0.001 0.001" />
                 </geometry>
                 <origin rpy="${pi/2} 0 0" xyz="${-body_length/2} ${body_width/2} ${-body_height/2}" />
@@ -47,12 +51,11 @@
             <collision>
                 <geometry>
-                    <mesh filename="package://workcell_description/meshes/Gripper.stl" scale="0.001 0.001 0.001"/>
+                    <mesh filename="package://workcell_description/meshes/Gripper.stl" scale="0.001 0.001 0.001" />
                 </geometry>
-                <origin rpy="0 0 0" xyz="0 0 0" />
+                <origin rpy="${pi/2} 0 0" xyz="${-body_length/2} ${body_width/2} ${-body_height/2}" />
             </collision>
-            <inertial>
-                <mass value="0.51" />
-                <inertia ixx="0.0007" iyy="0.0001" izz="0.0006" ixy="0.0" ixz="0.0" iyz="0.0" />
-            </inertial>
+            <xacro:inertial_box mass="0.5" x="${body_length}" y="${body_width}" z="${body_height}">
+                <origin rpy="${pi/2} 0 0" xyz="${-body_length/2} ${body_width/2} ${-body_height/2}" />
+            </xacro:inertial_box>
         </link>
         <!--Pincer block 1-->
@@ -60,5 +63,5 @@
             <visual>
                 <geometry>
-                    <mesh filename="package://workcell_description/meshes/Pincer_1.stl" scale="0.001 0.001 0.001"/>
+                    <mesh filename="package://workcell_description/meshes/Pincer_1.stl" scale="0.001 0.001 0.001" />
                 </geometry>
                 <origin rpy="${pi/2} 0 0" xyz="${-body_length/2} ${pincer_width/2} ${-body_height-pincer_height/2}" />
@@ -67,12 +70,11 @@
             <collision>
                 <geometry>
-                    <mesh filename="package://workcell_description/meshes/Pincer_1.stl" scale="0.001 0.001 0.001"/>
+                    <mesh filename="package://workcell_description/meshes/Pincer_1.stl" scale="0.001 0.001 0.001" />
                 </geometry>
                 <origin rpy="${pi/2} 0 0" xyz="${-body_length/2} ${pincer_width/2} ${-body_height-pincer_height/2}" />
             </collision>
-            <inertial>
-                <mass value="0.51" />
-                <inertia ixx="0.0007" iyy="0.0001" izz="0.0006" ixy="0.0" ixz="0.0" iyz="0.0" />
-            </inertial>
+            <xacro:inertial_box mass="0.1" x="${pincer_length}" y="${pincer_width}" z="${pincer_height}">
+                <origin rpy="${pi/2} 0 0" xyz="${-body_length/2} ${pincer_width/2} ${-body_height-pincer_height/2}" />
+            </xacro:inertial_box>
         </link>
         <!--Pincer block 2-->
@@ -80,5 +82,5 @@
             <visual>
                 <geometry>
-                    <mesh filename="package://workcell_description/meshes/Pincer_2.stl" scale="0.001 0.001 0.001"/>
+                    <mesh filename="package://workcell_description/meshes/Pincer_2.stl" scale="0.001 0.001 0.001" />
                 </geometry>
                 <origin rpy="${pi/2} 0 0" xyz="${-body_length/2} ${pincer_width/2} ${-body_height-pincer_height/2}" />
@@ -87,12 +89,11 @@
             <collision>
                 <geometry>
-                    <mesh filename="package://workcell_description/meshes/Pincer_2.stl" scale="0.001 0.001 0.001"/>
+                    <mesh filename="package://workcell_description/meshes/Pincer_2.stl" scale="0.001 0.001 0.001" />
                 </geometry>
                 <origin rpy="${pi/2} 0 0" xyz="${-body_length/2} ${pincer_width/2} ${-body_height-pincer_height/2}" />
             </collision>
-            <inertial>
-                <mass value="0.51" />
-                <inertia ixx="0.0007" iyy="0.0001" izz="0.0006" ixy="0.0" ixz="0.0" iyz="0.0" />
-            </inertial>
+            <xacro:inertial_box mass="0.1" x="${pincer_length}" y="${pincer_width}" z="${pincer_height}">
+                <origin rpy="${pi/2} 0 0" xyz="${-body_length/2} ${pincer_width/2} ${-body_height-pincer_height/2}" />
+            </xacro:inertial_box>
         </link>
         <!-- Virtual link for visualizytion and planning-->
@@ -109,7 +110,7 @@
             <origin xyz="0.0 0.0 ${body_height/2+pincer_height/2}" rpy="0.0 0.0 0.0" />
             <!-- the motion of the pincer is along the X axis -->
-            <axis xyz="1 0 0"/>
+            <axis xyz="1 0 0" />
             <!-- the motion of the pincer is limited to the half of the gripper body length -->
-            <limit lower="${-body_length/16}" upper="${body_length/16}" velocity="100" effort="100"/>
+            <limit lower="${-body_length/16}" upper="${body_length/16}" velocity="100" effort="100" />
         </joint>
         <joint name="shunk_egp50_pincer_2_joint" type="prismatic">
@@ -118,7 +119,7 @@
             <origin xyz="0.0 0.002 ${body_height/2+pincer_height/2}" rpy="0.0 0.0 0.0" />
             <!-- the motion of the pincer is along the X axis -->
-            <axis xyz="1 0 0"/>
+            <axis xyz="1 0 0" />
             <!-- the motion of the pincer is limited to the half of the gripper body length -->
-            <limit lower="${body_length/16}" upper="${-body_length/16}" velocity="100" effort="100"/>
+            <limit lower="${body_length/16}" upper="${-body_length/16}" velocity="100" effort="100" />
         </joint>
         <joint name="shunk_egp50_tip_joint" type="fixed">

File: workcell_description/urdf/workcell.urdf.xacro (robot description, xacro)
@@ -9,3 +9,4 @@
     <!-- loading camera from workcell_description package-->
     <xacro:include filename="$(find workcell_description)/urdf/camera.xacro" />
+    <xacro:include filename="$(find workcell_description)/urdf/gazebo_control.xacro" />
 </robot>
