Commit message: made a baseline urdf

File: workcell_description/urdf/gazebo_control.xacro (robot description, xacro)
@@ -3,18 +3,4 @@
     <!-- This plugin will publish the joint_states for the selected joints
             (which robot_state_publisher can then use to broadcast the approprate tf). -->
-    <gazebo>
-        <plugin name="gazebo_ros_joint_state_publisher"
-            filename="libgazebo_ros_joint_state_publisher.so">
-            <update_rate>200</update_rate>
-            <joint_name>shoulder_pan_joint</joint_name>
-            <joint_name>shoulder_lift_joint</joint_name>
-            <joint_name>elbow joint</joint_name>
-            <joint_name>wrist_1_joint</joint_name>
-            <joint_name>wrist_2_joint</joint_name>
-            <joint_name>wrist_3_joint</joint_name>
-            <joint_name>shunk_egp50_pincer_1_joint</joint_name>
-            <joint_name>shunk_egp50_pincer_2_joint</joint_name>
-        </plugin>
-    </gazebo>
     <!-- This plugin will read a JointTrajectory message from the /set_joint_trajectory topic
             and move the machine accordingly. -->

File: workcell_description/urdf/robot.xacro (robot description, xacro)
@@ -1,95 +1,104 @@
 <?xml version="1.0"?>
-<robot xmlns:xacro="http://www.ros.org/wiki/xacro">
-    <xacro:property name="robot_base_length" value="0.30" />
-    <xacro:property name="robot_base_width" value="0.52" />
-    <xacro:property name="robot_base_offset_length" value="0.45" />
-    <xacro:property name="robot_base_offset_width" value="0.02" />
-    <xacro:property name="robot_base_height" value="0.99" />
-    <xacro:property name="robotcell_length" value="1.44" />
-    <xacro:property name="robotcell_width" value="0.94" />
-    <xacro:property name="robotcell_height" value="1.16" />
-    <xacro:property name="shield_thickness" value="0.03" />
-    <joint name="robotcell_to_robot_joint" type="fixed">
-        <parent link="robotcell_link" />
-        <child link="base_link" />
-        <origin xyz="${robot_base_offset_length} ${-robot_base_offset_width} ${robot_base_height}" rpy="0 0 ${-pi}" />
-    </joint>
-    <!-- robot name parameter -->
-    <xacro:arg name="name" default="ur" />
-    <!-- import main macro -->
-    <xacro:include filename="$(find ur_description)/urdf/ur_macro.xacro" />
-    <!-- possible 'ur_type' values: ur3, ur3e, ur5, ur5e, ur10, ur10e, ur16e -->
-    <!-- the default value should raise an error in case this was called without defining the type -->
-    <xacro:arg name="ur_type" default="ur5e" />
-    <!-- parameters -->
-    <xacro:arg name="prefix" default="" />
-    <xacro:arg name="joint_limit_params" default="$(find ur_description)/config/$(arg ur_type)/joint_limits.yaml" />
-    <xacro:arg name="kinematics_params" default="$(find ur_description)/config/$(arg ur_type)/default_kinematics.yaml" />
-    <xacro:arg name="physical_params" default="$(find ur_description)/config/$(arg ur_type)/physical_parameters.yaml" />
-    <xacro:arg name="visual_params" default="$(find ur_description)/config/$(arg ur_type)/visual_parameters.yaml" />
-    <xacro:arg name="transmission_hw_interface" default="" />
-    <xacro:arg name="safety_limits" default="false" />
-    <xacro:arg name="safety_pos_margin" default="0.15" />
-    <xacro:arg name="safety_k_position" default="20" />
-    <!-- ros2_control related parameters -->
-    <xacro:arg name="headless_mode" default="false" />
-    <xacro:arg name="robot_ip" default="0.0.0.0" />
-    <xacro:arg name="script_filename" default="" />
-    <xacro:arg name="output_recipe_filename" default="" />
-    <xacro:arg name="input_recipe_filename" default="" />
-    <!--   tool communication related parameters-->
-    <xacro:arg name="use_tool_communication" default="false" />
-    <xacro:arg name="tool_voltage" default="24" />
-    <xacro:arg name="tool_parity" default="0" />
-    <xacro:arg name="tool_baud_rate" default="115200" />
-    <xacro:arg name="tool_stop_bits" default="1" />
-    <xacro:arg name="tool_rx_idle_chars" default="1.5" />
-    <xacro:arg name="tool_tx_idle_chars" default="3.5" />
-    <xacro:arg name="tool_device_name" default="/tmp/ttyUR" />
-    <xacro:arg name="tool_tcp_port" default="54321" />
-    <!-- Simulation parameters -->
-    <xacro:arg name="use_fake_hardware" default="false" />
-    <xacro:arg name="fake_sensor_commands" default="false" />
-    <xacro:arg name="sim_gazebo" default="true" />
-    <xacro:arg name="sim_ignition" default="true" />
-    <xacro:arg name="simulation_controllers" default="" />
-    <!-- initial position for simulations (Fake Hardware, Gazebo, Ignition) -->
-    <xacro:arg name="initial_positions_file" default="$(find ur_description)/config/initial_positions.yaml" />
-    <!-- convert to property to use substitution in function -->
-    <xacro:property name="initial_positions_file" default="$(arg initial_positions_file)" />
-    <!-- arm -->
-    <xacro:ur_robot
-        name="$(arg name)"
-        prefix="$(arg prefix)"
-        parent="world"
-        joint_limits_parameters_file="$(arg joint_limit_params)"
-        kinematics_parameters_file="$(arg kinematics_params)"
-        physical_parameters_file="$(arg physical_params)"
-        visual_parameters_file="$(arg visual_params)"
-        transmission_hw_interface="$(arg transmission_hw_interface)"
-        safety_limits="$(arg safety_limits)"
-        safety_pos_margin="$(arg safety_pos_margin)"
-        safety_k_position="$(arg safety_k_position)"
-        use_fake_hardware="$(arg use_fake_hardware)"
-        fake_sensor_commands="$(arg fake_sensor_commands)"
-        sim_gazebo="$(arg sim_gazebo)"
-        sim_ignition="$(arg sim_ignition)"
-        headless_mode="$(arg headless_mode)"
-        initial_positions="${load_yaml(initial_positions_file)}"
-        use_tool_communication="$(arg use_tool_communication)"
-        tool_voltage="$(arg tool_voltage)"
-        tool_parity="$(arg tool_parity)"
-        tool_baud_rate="$(arg tool_baud_rate)"
-        tool_stop_bits="$(arg tool_stop_bits)"
-        tool_rx_idle_chars="$(arg tool_rx_idle_chars)"
-        tool_tx_idle_chars="$(arg tool_tx_idle_chars)"
-        tool_device_name="$(arg tool_device_name)"
-        tool_tcp_port="$(arg tool_tcp_port)"
-        robot_ip="$(arg robot_ip)"
-        script_filename="$(arg script_filename)"
-        output_recipe_filename="$(arg output_recipe_filename)"
-        input_recipe_filename="$(arg input_recipe_filename)"
-    >
-        <origin xyz="0 0 0" rpy="0 0 0" /> <!-- position robot in the robotcell -->
-    </xacro:ur_robot>
+<robot xmlns:xacro="http://wiki.ros.org/xacro" name="ur5e">
+   <!-- robot name parameter -->
+   <xacro:arg name="name" default="ur5e"/>
+   <!-- import main macro -->
+   <xacro:include filename="$(find ur_description)/urdf/ur_macro.xacro"/>
+   <!-- possible 'ur_type' values: ur3, ur3e, ur5, ur5e, ur10, ur10e, ur16e -->
+   <!-- the default value should raise an error in case this was called without defining the type -->
+   <xacro:arg name="ur_type" default="ur5e"/>
+   <!-- parameters -->
+   <xacro:arg name="prefix" default="" />
+   <xacro:arg name="joint_limit_params" default="$(find ur_description)/config/$(arg ur_type)/joint_limits.yaml"/>
+   <xacro:arg name="kinematics_params" default="$(find ur_description)/config/$(arg ur_type)/default_kinematics.yaml"/>
+   <xacro:arg name="physical_params" default="$(find ur_description)/config/$(arg ur_type)/physical_parameters.yaml"/>
+   <xacro:arg name="visual_params" default="$(find ur_description)/config/$(arg ur_type)/visual_parameters.yaml"/>
+   <xacro:arg name="transmission_hw_interface" default=""/>
+   <xacro:arg name="safety_limits" default="false"/>
+   <xacro:arg name="safety_pos_margin" default="0.15"/>
+   <xacro:arg name="safety_k_position" default="20"/>
+   <!-- ros2_control related parameters -->
+   <xacro:arg name="headless_mode" default="false" />
+   <xacro:arg name="robot_ip" default="0.0.0.0" />
+   <xacro:arg name="script_filename" default=""/>
+   <xacro:arg name="output_recipe_filename" default=""/>
+   <xacro:arg name="input_recipe_filename" default=""/>
+   <!--   tool communication related parameters-->
+   <xacro:arg name="use_tool_communication" default="false" />
+   <xacro:arg name="tool_voltage" default="24" />
+   <xacro:arg name="tool_parity" default="0" />
+   <xacro:arg name="tool_baud_rate" default="115200" />
+   <xacro:arg name="tool_stop_bits" default="1" />
+   <xacro:arg name="tool_rx_idle_chars" default="1.5" />
+   <xacro:arg name="tool_tx_idle_chars" default="3.5" />
+   <xacro:arg name="tool_device_name" default="/tmp/ttyUR" />
+   <xacro:arg name="tool_tcp_port" default="54321" />
+     <!-- Simulation parameters -->
+   <xacro:arg name="use_fake_hardware" default="false" />
+   <xacro:arg name="fake_sensor_commands" default="false" />
+   <xacro:arg name="sim_gazebo" default="false" />
+   <xacro:arg name="sim_ignition" default="false" />
+   <xacro:arg name="simulation_controllers" default="" />
+   <!-- initial position for simulations (Fake Hardware, Gazebo, Ignition) -->
+   <xacro:arg name="initial_positions_file" default="$(find ur_description)/config/initial_positions.yaml"/>
+   <!-- convert to property to use substitution in function -->
+   <xacro:property name="initial_positions_file" default="$(arg initial_positions_file)"/>
+   <!-- create link fixed to the "world" -->
+   <link name="world" />
+   <!-- arm -->
+   <xacro:ur_robot
+     name="$(arg name)"
+     prefix="$(arg prefix)"
+     parent="world"
+     joint_limits_parameters_file="$(arg joint_limit_params)"
+     kinematics_parameters_file="$(arg kinematics_params)"
+     physical_parameters_file="$(arg physical_params)"
+     visual_parameters_file="$(arg visual_params)"
+     transmission_hw_interface="$(arg transmission_hw_interface)"
+     safety_limits="$(arg safety_limits)"
+     safety_pos_margin="$(arg safety_pos_margin)"
+     safety_k_position="$(arg safety_k_position)"
+     use_fake_hardware="$(arg use_fake_hardware)"
+     fake_sensor_commands="$(arg fake_sensor_commands)"
+     sim_gazebo="$(arg sim_gazebo)"
+     sim_ignition="$(arg sim_ignition)"
+     headless_mode="$(arg headless_mode)"
+     initial_positions="${load_yaml(initial_positions_file)}"
+     use_tool_communication="$(arg use_tool_communication)"
+     tool_voltage="$(arg tool_voltage)"
+     tool_parity="$(arg tool_parity)"
+     tool_baud_rate="$(arg tool_baud_rate)"
+     tool_stop_bits="$(arg tool_stop_bits)"
+     tool_rx_idle_chars="$(arg tool_rx_idle_chars)"
+     tool_tx_idle_chars="$(arg tool_tx_idle_chars)"
+     tool_device_name="$(arg tool_device_name)"
+     tool_tcp_port="$(arg tool_tcp_port)"
+     robot_ip="$(arg robot_ip)"
+     script_filename="$(arg script_filename)"
+     output_recipe_filename="$(arg output_recipe_filename)"
+     input_recipe_filename="$(arg input_recipe_filename)"
+     >
+     <origin xyz="0 0 0" rpy="0 0 0" />          <!-- position robot in the world -->
+   </xacro:ur_robot>
+   <xacro:if value="$(arg sim_gazebo)">
+    <!-- Gazebo plugins -->
+    <gazebo reference="world">
+    </gazebo>
+    <gazebo>
+      <plugin filename="libgazebo_ros2_control.so" name="gazebo_ros2_control">
+        <parameters>$(arg simulation_controllers)</parameters>
+      </plugin>
+    </gazebo>
+  </xacro:if>
+  <xacro:if value="$(arg sim_ignition)">
+    <!-- Gazebo plugins -->
+    <gazebo reference="world">
+    </gazebo>
+    <gazebo>
+      <plugin filename="libign_ros2_control-system.so" name="ign_ros2_control::IgnitionROS2ControlPlugin">
+        <parameters>$(arg simulation_controllers)</parameters>
+        <controller_manager_node_name>$(arg prefix)controller_manager</controller_manager_node_name>
+      </plugin>
+    </gazebo>
+  </xacro:if>
 </robot>

File: workcell_description/urdf/robot_cell_clone.xacro (robot description, xacro)
@@ -12,5 +12,4 @@
         <color rgba="0.6 0.8 0.8 1" />
     </material>
-    <link name="world"></link>
     <link name="robotcell_link">
         <origin xyz="0 0 0" rpy="0 0 0" />
@@ -104,9 +103,4 @@
         </xacro:inertial_box>
     </link>
-    <joint name="world_to_robotcell_joint" type="fixed">
-        <parent link="world" />
-        <child link="robotcell_link" />
-        <origin xyz="0 0 0" rpy="0 0 0" />
-    </joint>
     <joint name="robotcell_joint_to_front" type="fixed">
         <parent link="robotcell_link" />

File: workcell_description/urdf/shunk_egp50.xacro (robot description, xacro)
@@ -105,5 +105,5 @@
             <origin xyz="0.0 0.0 ${base_length+body_height/2}" rpy="0.0 0.0 0.0" />
         </joint>
-        <joint name="shunk_egp50_pincer_1_joint" type="prismatic">
+        <joint name="shunk_egp50_pincer_1_joint" type="fixed">
             <parent link="shunk_egp50_body_link" />
             <child link="shunk_egp50_pincer_1_link" />
@@ -114,5 +114,5 @@
             <limit lower="${-body_length/16}" upper="${body_length/16}" velocity="100" effort="100" />
         </joint>
-        <joint name="shunk_egp50_pincer_2_joint" type="prismatic">
+        <joint name="shunk_egp50_pincer_2_joint" type="fixed">
             <parent link="shunk_egp50_body_link" />
             <child link="shunk_egp50_pincer_2_link" />

File: workcell_description/urdf/workcell.urdf (robot description, URDF)
Before this commit: robot ur5e_workcell, 26 links, 26 joints
Links:
- link base_link_inertia: geometry collision mesh filename=file:///home/ragesh/ur_ws/install/ur_description/share/ur_d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; visual mesh filename=file:///home/ragesh/ur_ws/install/ur_description/share/ur_d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
- link forearm_link: geometry collision mesh filename=file:///home/ragesh/ur_ws/install/ur_description/share/ur_d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; visual mesh filename=file:///home/ragesh/ur_ws/install/ur_description/share/ur_d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
- link shoulder_link: geometry collision mesh filename=file:///home/ragesh/ur_ws/install/ur_description/share/ur_d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; visual mesh filename=file:///home/ragesh/ur_ws/install/ur_description/share/ur_d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
- link upper_arm_link: geometry collision mesh filename=file:///home/ragesh/ur_ws/install/ur_description/share/ur_d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; visual mesh filename=file:///home/ragesh/ur_ws/install/ur_description/share/ur_d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
- link wrist_1_link: geometry collision mesh filename=file:///home/ragesh/ur_ws/install/ur_description/share/ur_d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; visual mesh filename=file:///home/ragesh/ur_ws/install/ur_description/share/ur_d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
- link wrist_2_link: geometry collision mesh filename=file:///home/ragesh/ur_ws/install/ur_description/share/ur_d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; visual mesh filename=file:///home/ragesh/ur_ws/install/ur_description/share/ur_d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
- link wrist_3_link: geometry collision mesh filename=file:///home/ragesh/ur_ws/install/ur_description/share/ur_d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; visual mesh filename=file:///home/ragesh/ur_ws/install/ur_description/share/ur_d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

File: workcell_description/urdf/workcell.urdf.xacro (robot description, xacro)
@@ -1,13 +1,25 @@
 <?xml version="1.0"?>
 <robot xmlns:xacro="http://www.ros.org/wiki/xacro" name="ur5e_workcell">
-    <!-- loading robotcell from workcell_description package-->
-    <xacro:include filename="$(find workcell_description)/urdf/robot_cell_clone.xacro" />
     <!-- loading robot  from workcell_description package-->
     <xacro:include filename="$(find workcell_description)/urdf/robot.xacro" />
-    <!-- loading gripper from workcell_description package-->
-    <xacro:include filename="$(find workcell_description)/urdf/gripper.xacro" />
-    <!-- loading camera from workcell_description package-->
-    <xacro:include filename="$(find workcell_description)/urdf/camera.xacro" />
-    <!-- loading gazebo plugins-->
-    <xacro:include filename="$(find workcell_description)/urdf/gazebo_control.xacro" />
+    <xacro:include filename="$(find workcell_description)/urdf/shunk_egp50.xacro" />
+    <xacro:include filename="$(find workcell_description)/urdf/robot_cell_clone.xacro"/>
+    <xacro:property name="gripper_name" value="shunk_egp50" />
+    <xacro:schunk_egp50 />
+    <joint name="robot_to_gripper_joint" type="fixed">
+        <parent link="tool0" />
+        <child link="${gripper_name}_base_link" />
+        <origin xyz="0.0 0.0 0.0" rpy="0.0 0.0 0.0" />
+    </joint>
+    <joint name="base_link_to_robotcell_joint" type="fixed">
+        <parent link="base_link" />
+        <child link="robotcell_link" />
+        <origin xyz="0 0 ${-robot_base_height}" rpy="0 0 0" />
+    </joint>
+<!--     <joint name="robotcell_to_base_link_joint" type="fixed">
+        <parent link="robotcell_link" />
+        <child link="base_link" />
+        <origin xyz="0 0 0" rpy="0 0 0" />
+    </joint>
+ -->
 </robot>
