Commit message: launch filestill not fixed

File: workcell_description/urdf/robot_cell_clone.xacro (robot description, xacro)
@@ -20,5 +20,5 @@
             <origin rpy="0 0 0" xyz="0 0 0" />
             <geometry>
-                <box size="${robotcell_length} ${shield_thickness} ${shield_thickness}" />
+                <box size="${robotcell_length} ${shield_thickness} ${robotcell_height}" />
             </geometry>
             <material name="gray"/>

File: workcell_description/urdf/workcell.urdf (robot description, URDF)
Before this commit: robot ur5e_workcell, 26 links, 26 joints
Links:
- link base_link_inertia: geometry collision mesh filename=package://workcell_description/meshes/collision/base.stl; visual mesh filename=package://workcell_description/meshes/visual/base.dae
- link forearm_link: geometry collision mesh filename=package://workcell_description/meshes/collision/forearm.stl; visual mesh filename=package://workcell_description/meshes/visual/forearm.dae
- link shield_front: geometry collision box size=1.44 0.03 1.16
- link shoulder_link: geometry collision mesh filename=package://workcell_description/meshes/collision/shoulder.stl; visual mesh filename=package://workcell_description/meshes/visual/shoulder.dae
- link upper_arm_link: geometry collision mesh filename=package://workcell_description/meshes/collision/upperarm.stl; visual mesh filename=package://workcell_description/meshes/visual/upperarm.dae
- link wrist_1_link: geometry collision mesh filename=package://workcell_description/meshes/collision/wrist1.stl; visual mesh filename=package://workcell_description/meshes/visual/wrist1.dae
- link wrist_2_link: geometry collision mesh filename=package://workcell_description/meshes/collision/wrist2.stl; visual mesh filename=package://workcell_description/meshes/visual/wrist2.dae
- link wrist_3_link: geometry collision mesh filename=package://workcell_description/meshes/collision/wrist3.stl; visual mesh filename=package://workcell_description/meshes/visual/wrist3.dae

Commit message: urdf refactored & tested in the vfeld D

File: workcell_description/urdf/robot_cell_clone.xacro (robot description, xacro)
@@ -2,6 +2,6 @@
 <robot xmlns:xacro="http://www.ros.org/wiki/xacro">
     <xacro:include filename="inertial_macros.xacro"/>
-    <xacro:property name="robot_base_length" value="0.45" />
-    <xacro:property name="robot_base_width" value="0.52" />
+    <xacro:property name="robot_center_offset_length" value="0.42" />
+    <xacro:property name="robot_center_offset_width" value="0.02" />
     <xacro:property name="robot_base_height" value="0.99" />
     <xacro:property name="robotcell_length" value="1.44" />
@@ -12,8 +12,5 @@
         <color rgba="0.6 0.8 0.8 1" />
     </material>
-    <link name="robotcell_link">
-        <origin xyz="0 0 0" rpy="0 0 0" />
-    </link>
-    <link name="shield_front">
+    <link name="shield_front_link">
         <collision>
             <origin rpy="0 0 0" xyz="0 0 0" />
@@ -27,5 +24,5 @@
         </xacro:inertial_box>
     </link>
-    <link name="shield_rear">
+    <link name="shield_rear_link">
         <visual>
             <origin rpy="0 0 0" xyz="0 0 0" />
@@ -46,5 +43,5 @@
         </xacro:inertial_box>
     </link>
-    <link name="shield_left">
+    <link name="shield_right_link">
         <visual>
             <origin rpy="0 0 0" xyz="0 0 0" />
@@ -65,5 +62,5 @@
         </xacro:inertial_box>
     </link>
-    <link name="shield_right">
+    <link name="shield_left_link">
         <visual>
             <origin rpy="0 0 0" xyz="0 0 0" />
@@ -84,5 +81,5 @@
         </xacro:inertial_box>
     </link>
-    <link name="robotcell_base">
+    <link name="robotcell_base_link">
         <visual>
             <origin rpy="0 0 0" xyz="0 0 ${robot_base_height/2}" />
@@ -103,28 +100,23 @@
         </xacro:inertial_box>
     </link>
-    <joint name="robotcell_joint_to_front" type="fixed">
-        <parent link="robotcell_link" />
-        <child link="shield_front" />
+    <joint name="robotcell_base_to_front_joint" type="fixed">
+        <parent link="robotcell_base_link" />
+        <child link="shield_front_link" />
         <origin xyz="0 ${robotcell_width/2-shield_thickness/2} ${robot_base_height+robotcell_height/2}" rpy="0 0 0" />
     </joint>
-    <joint name="robotcell_joint_to_rear" type="fixed">
-        <parent link="robotcell_link" />
-        <child link="shield_rear" />
+    <joint name="robotcell_base_to_rear" type="fixed">
+        <parent link="robotcell_base_link" />
+        <child link="shield_rear_link" />
         <origin xyz="0 ${-robotcell_width/2+shield_thickness/2} ${robot_base_height+robotcell_height/2}" rpy="0 0 0" />
     </joint>
-    <joint name="robotcell_joint_to_left" type="fixed">
-        <parent link="robotcell_link" />
-        <child link="shield_left" />
+    <joint name="robotcell_base_to_left" type="fixed">
+        <parent link="robotcell_base_link" />
+        <child link="shield_left_link" />
         <origin xyz="${-robotcell_length/2+shield_thickness/2} 0 ${robot_base_height+robotcell_height/2}" rpy="0 0 0" />
     </joint>
-    <joint name="robotcell_joint_to_right" type="fixed">
-        <parent link="robotcell_link" />
-        <child link="shield_right" />
+    <joint name="robotcell_jbase_to_right" type="fixed">
+        <parent link="robotcell_base_link" />
+        <child link="shield_right_link" />
         <origin xyz="${robotcell_length/2-shield_thickness/2} 0 ${robot_base_height+robotcell_height/2}" rpy="0 0 0" />
     </joint>
-    <joint name="robotcell_joint_to_robotcell_base" type="fixed">
-        <parent link="robotcell_link" />
-        <child link="robotcell_base" />
-        <origin xyz="0 0 0" rpy="0 0 0" />
-    </joint>
 </robot>

File: workcell_description/urdf/workcell.urdf (robot description, URDF)
Before this commit: robot ur5e_workcell, 26 links, 26 joints
Links:
- removed link camera_bottom_screw_frame
- removed link camera_link
- link base_link_inertia: geometry collision mesh filename=package://ur_description/meshes/ur5e/collision/base.stl; visual mesh filename=package://ur_description/meshes/ur5e/visual/base.dae
- link forearm_link: geometry collision mesh filename=package://ur_description/meshes/ur5e/collision/forearm.stl; visual mesh filename=package://ur_description/meshes/ur5e/visual/forearm.dae
- link shoulder_link: geometry collision mesh filename=package://ur_description/meshes/ur5e/collision/shoulder.stl; visual mesh filename=package://ur_description/meshes/ur5e/visual/shoulder.dae
- link upper_arm_link: geometry collision mesh filename=package://ur_description/meshes/ur5e/collision/upperarm.stl; visual mesh filename=package://ur_description/meshes/ur5e/visual/upperarm.dae
- link wrist_1_link: geometry collision mesh filename=package://ur_description/meshes/ur5e/collision/wrist1.stl; visual mesh filename=package://ur_description/meshes/ur5e/visual/wrist1.dae
- link wrist_2_link: geometry collision mesh filename=package://ur_description/meshes/ur5e/collision/wrist2.stl; visual mesh filename=package://ur_description/meshes/ur5e/visual/wrist2.dae
- link wrist_3_link: geometry collision mesh filename=package://ur_description/meshes/ur5e/collision/wrist3.stl; visual mesh filename=package://ur_description/meshes/ur5e/visual/wrist3.dae
Joints:
- removed joint camera_joint
- removed joint camera_link_joint
- removed joint robotcell_to_robot_joint
- removed joint world_to_robotcell_joint
- added joint world_to_robot_cell_joint: type fixed, parent world, child robotcell_link, origin xyz=0 0 0 rpy=0 0 0
- joint base_joint: origin xyz=0 0 0 rpy=0 0 0 -> xyz=0 0 0.495 rpy=0 0 0; parent world -> robotcell_base
- joint shunk_egp50_pincer_1_joint: type prismatic -> fixed
- joint shunk_egp50_pincer_2_joint: type prismatic -> fixed

File: workcell_description/urdf/workcell.urdf.xacro (robot description, xacro)
@@ -2,9 +2,90 @@
 <robot xmlns:xacro="http://www.ros.org/wiki/xacro" name="ur5e_workcell">
     <!-- loading robot  from workcell_description package-->
-    <xacro:include filename="$(find workcell_description)/urdf/robot.xacro" />
     <xacro:include filename="$(find workcell_description)/urdf/shunk_egp50.xacro" />
-    <xacro:include filename="$(find workcell_description)/urdf/robot_cell_clone.xacro"/>
+    <xacro:include filename="$(find workcell_description)/urdf/robot_cell_clone.xacro" />
+    <xacro:include filename="$(find ur_description)/urdf/ur_macro.xacro" />
+    <xacro:arg name="name" default="ur5e" />
+    <xacro:arg name="ur_type" default="ur5e" />
+    <xacro:arg name="prefix" default="" />
+    <xacro:arg name="joint_limit_params" default="$(find ur_description)/config/$(arg ur_type)/joint_limits.yaml" />
+    <xacro:arg name="kinematics_params" default="$(find ur_description)/config/$(arg ur_type)/default_kinematics.yaml" />
+    <xacro:arg name="physical_params" default="$(find ur_description)/config/$(arg ur_type)/physical_parameters.yaml" />
+    <xacro:arg name="visual_params" default="$(find ur_description)/config/$(arg ur_type)/visual_parameters.yaml" />
+    <xacro:arg name="transmission_hw_interface" default="" />
+    <xacro:arg name="safety_limits" default="false" />
+    <xacro:arg name="safety_pos_margin" default="0.15" />
+    <xacro:arg name="safety_k_position" default="20" />
+    <xacro:arg name="headless_mode" default="false" />
+    <xacro:arg name="robot_ip" default="0.0.0.0" />
+    <xacro:arg name="script_filename" default="" />
+    <xacro:arg name="output_recipe_filename" default="" />
+    <xacro:arg name="input_recipe_filename" default="" />
+    <xacro:arg name="use_tool_communication" default="false" />
+    <xacro:arg name="tool_voltage" default="24" />
+    <xacro:arg name="tool_parity" default="0" />
+    <xacro:arg name="tool_baud_rate" default="115200" />
+    <xacro:arg name="tool_stop_bits" default="1" />
+    <xacro:arg name="tool_rx_idle_chars" default="1.5" />
+    <xacro:arg name="tool_tx_idle_chars" default="3.5" />
+    <xacro:arg name="tool_device_name" default="/tmp/ttyUR" />
+    <xacro:arg name="tool_tcp_port" default="54321" />
+    <xacro:arg name="use_fake_hardware" default="false" />
+    <xacro:arg name="fake_sensor_commands" default="false" />
+    <xacro:arg name="sim_gazebo" default="false" />
+    <xacro:arg name="sim_ignition" default="false" />
+    <xacro:arg name="simulation_controllers" default="" />
+    <xacro:arg name="initial_positions_file" default="$(find ur_description)/config/initial_positions.yaml" />
     <xacro:property name="gripper_name" value="shunk_egp50" />
+    <xacro:property name="initial_positions_file" default="$(arg initial_positions_file)" />
     <xacro:schunk_egp50 />
+    <xacro:ur_robot
+        name="$(arg name)"
+        prefix="$(arg prefix)"
+        parent="robotcell_base_link"
+        joint_limits_parameters_file="$(arg joint_limit_params)"
+        kinematics_parameters_file="$(arg kinematics_params)"
+        physical_parameters_file="$(arg physical_params)"
+        visual_parameters_file="$(arg visual_params)"
+        transmission_hw_interface="$(arg transmission_hw_interface)"
+        safety_limits="$(arg safety_limits)"
+        safety_pos_margin="$(arg safety_pos_margin)"
+        safety_k_position="$(arg safety_k_position)"
+        use_fake_hardware="$(arg use_fake_hardware)"
+        fake_sensor_commands="$(arg fake_sensor_commands)"
+        sim_gazebo="$(arg sim_gazebo)"
+        sim_ignition="$(arg sim_ignition)"
+        headless_mode="$(arg headless_mode)"
+        initial_positions="${load_yaml(initial_positions_file)}"
+        use_tool_communication="$(arg use_tool_communication)"
+        tool_voltage="$(arg tool_voltage)"
+        tool_parity="$(arg tool_parity)"
+        tool_baud_rate="$(arg tool_baud_rate)"
+        tool_stop_bits="$(arg tool_stop_bits)"
+        tool_rx_idle_chars="$(arg tool_rx_idle_chars)"
+        tool_tx_idle_chars="$(arg tool_tx_idle_chars)"
+        tool_device_name="$(arg tool_device_name)"
+        tool_tcp_port="$(arg tool_tcp_port)"
+        robot_ip="$(arg robot_ip)"
+        script_filename="$(arg script_filename)"
+        output_recipe_filename="$(arg output_recipe_filename)"
+        input_recipe_filename="$(arg input_recipe_filename)"
+    >
+        <origin xyz="${robot_center_offset_length} ${robot_center_offset_width} ${robot_base_height}" rpy="0 0 ${pi/2}" /> <!-- position robot in the world -->
+    </xacro:ur_robot>
+    <xacro:if value="$(arg sim_gazebo)">
+        <!-- Gazebo plugins -->
+        <gazebo reference="world"></gazebo>
+        <gazebo>
+            <plugin filename="libgazebo_ros2_control.so" name="gazebo_ros2_control">
+                <parameters>$(arg simulation_controllers)</parameters>
+            </plugin>
+        </gazebo>
+    </xacro:if>
+    <link name="world" />
+    <joint name="world_to_robot_cell_joint" type="fixed">
+        <parent link="world" />
+        <child link="robotcell_base_link" />
+        <origin xyz="0 0 0" rpy="0 0 0" />
+    </joint>
     <joint name="robot_to_gripper_joint" type="fixed">
         <parent link="tool0" />
@@ -12,14 +93,3 @@
         <origin xyz="0.0 0.0 0.0" rpy="0.0 0.0 0.0" />
     </joint>
-    <joint name="base_link_to_robotcell_joint" type="fixed">
-        <parent link="base_link" />
-        <child link="robotcell_link" />
-        <origin xyz="0 0 ${-robot_base_height}" rpy="0 0 0" />
-    </joint>
-<!--     <joint name="robotcell_to_base_link_joint" type="fixed">
-        <parent link="robotcell_link" />
-        <child link="base_link" />
-        <origin xyz="0 0 0" rpy="0 0 0" />
-    </joint>
- -->
 </robot>
