Commit message: fixed issues with urdf files

File: workcell_description/urdf/workcell.urdf.xacro (robot description, xacro)
@@ -1,70 +1,11 @@
 <?xml version="1.0"?>
-<robot name="ur5e_workcell" xmlns:xacro="http://www.ros.org/wiki/xacro">
-    <!-- loading ur5e xacro from ur_description package-->
-    <xacro:include filename="$(find ur_description)/urdf/ur_macro.xacro" />
-    <!-- loading schunk_egp50 xacro from workcell_description package-->
-    <xacro:include filename="$(find workcell_description)/urdf/gripper.urdf.xacro" />
-    <!-- loading realsense xacro from realsense2_description package-->
-    <xacro:include filename="$(find realsense2_description)/urdf/_d435.urdf.xacro" />
-    <!-- intel real sense -->
-    <xacro:arg name="use_nominal_extrinsics" default="false"/>
-    <xacro:arg name="add_plug" default="false" />
-    <xacro:arg name="use_mesh" default="true" />
-    <!-- ur5e -->
-    <xacro:arg name="ur_type" default="ur5"/>
-    <xacro:arg name="use_fake_hardware" default="true"/>
-    <xacro:arg name="fake_sensor_commands" default="true"/>
-    <!-- Instantiate arm -->
-    <xacro:ur_robot
-        prefix=""
-        joint_limits_parameters_file="$(find ur_description)/config/$(arg ur_type)/joint_limits.yaml"
-        kinematics_parameters_file="$(find ur_description)/config/$(arg ur_type)/default_kinematics.yaml"
-        physical_parameters_file="$(find ur_description)/config/$(arg ur_type)/physical_parameters.yaml"
-        visual_parameters_file="$(find ur_description)/config/$(arg ur_type)/visual_parameters.yaml"
-        use_fake_hardware="$(arg use_fake_hardware)"
-        fake_sensor_commands="$(arg fake_sensor_commands)"/>
-    <!-- Instantiate gripper -->
-    <xacro:schunk_egp50 />
-    <!-- Instantiate realsense camera -->
-    <xacro:sensor_d435
-        parent="base_link"
-        name="camera"
-        use_nominal_extrinsics="$(arg use_nominal_extrinsics)"
-        add_plug="$(arg add_plug)"
-        use_mesh="$(arg use_mesh)">
-        <origin xyz="0.1 0 0" rpy="0 0 0"/>
-    </xacro:sensor_d435>
-    <link name="world" />
-    <link name="robotcell">
-        <visual>
-            <origin rpy="0.0 0 0" xyz="0 0 0" />
-            <geometry>
-                <mesh filename="package://workcell_description/meshes/Robotcell.stl" />
-            </geometry>
-        </visual>
-    </link>
-    <link name="camera"/>
-    <joint name="world_to_robotcell" type="fixed">
-        <parent link="world" />
-        <child link="robotcell" />
-        <origin xyz="-0.25 -0.25 0" rpy="0 0 0" />
-    </joint>
-    <joint name="robotcell_to_robot" type="fixed">
-        <parent link="robotcell" />
-        <child link="base_link" />
-        <origin xyz="0 0 0" rpy="0 0 0" />
-    </joint>
-    <joint name="robot_to_gripper" type="fixed">
-        <parent link="wrist_3_link" />
-        <child link="egp50_base_link" />
-        <origin xyz="0.0 0.0 0.0" rpy="0.0 0.0 0.0" />
-    </joint>
-    <joint name="base_link_to_camera" type="fixed">
-        <parent link="base_link" />
-        <child link="camera" />
-        <origin xyz="0.25 0.25 0.5" rpy="0 -3.14 0" />
-    </joint>
-    <gazebo>
-        <plugin name="ros_control" filename="libgazebo_ros_control.so"></plugin>
-    </gazebo>
+<robot xmlns:xacro="http://www.ros.org/wiki/xacro" name="ur5e_workcell">
+    <!-- loading robotcell from workcell_description package-->
+    <xacro:include filename="$(find workcell_description)/urdf/robotcell.xacro" />
+    <!-- loading robot  from workcell_description package-->
+    <xacro:include filename="$(find workcell_description)/urdf/robot.xacro" />
+    <!-- loading gripper from workcell_description package-->
+    <xacro:include filename="$(find workcell_description)/urdf/gripper.xacro" />
+    <!-- loading camera from workcell_description package-->
+    <xacro:include filename="$(find workcell_description)/urdf/camera.xacro" />
 </robot>

Commit message: added camera component to urdf

File: workcell_description/urdf/workcell.urdf.xacro (robot description, xacro)
@@ -5,4 +5,5 @@
     <xacro:include filename="$(find workcell_description)/urdf/robot_cell_clone.xacro" />
     <xacro:include filename="$(find ur_description)/urdf/ur_macro.xacro" />
+    <xacro:include filename="$(find realsense2_description)/urdf/_d435.urdf.xacro" />
     <xacro:arg name="name" default="ur5e" />
     <xacro:arg name="ur_type" default="ur5e" />
@@ -36,4 +37,7 @@
     <xacro:arg name="simulation_controllers" default="" />
     <xacro:arg name="initial_positions_file" default="$(find ur_description)/config/initial_positions.yaml" />
+    <xacro:arg name="use_nominal_extrinsics" default="false" />
+    <xacro:arg name="add_plug" default="false" />
+    <xacro:arg name="use_mesh" default="true" />
     <xacro:property name="gripper_name" value="shunk_egp50" />
     <xacro:property name="initial_positions_file" default="$(arg initial_positions_file)" />
@@ -93,3 +97,10 @@
         <origin xyz="0.0 0.0 0.0" rpy="0.0 0.0 0.0" />
     </joint>
+    <xacro:sensor_d435
+        parent="robotcell_base_link"
+        use_nominal_extrinsics="$(arg use_nominal_extrinsics)"
+        add_plug="$(arg add_plug)"
+        use_mesh="$(arg use_mesh)">
+        <origin xyz="-0.285 0 ${robotcell_height+robot_base_height-shield_thickness}" rpy="${-pi/2} ${pi/2} 0" />
+    </xacro:sensor_d435>
 </robot>
