Commit message: back up repo

File: ur5e_cell_description/urdf/shunk_egp50.xacro (robot description, xacro)
@@ -8,5 +8,5 @@
         <xacro:property name="body_width" value="0.03" />
         <xacro:property name="body_height" value="0.0866" />
-        <xacro:property name="body_height_max" value="0.01044" />
+        <xacro:property name="body_height_max" value="0.1044" />
         <xacro:property name="pincer_height" value="0.014" />
         <xacro:property name="pincer_length" value="0.050" />
