Commit message: updated after robot testing in vfeld

File: ur5e_cell_description/urdf/workcell.urdf.xacro (robot description, xacro)
@@ -3,14 +3,15 @@
     <!-- loading robot  from ur5e_cell_description package-->
     <xacro:include filename="$(find ur5e_cell_description)/urdf/shunk_egp50.xacro" />
-    <!-- <xacro:include filename="$(find ur5e_cell_description)/urdf/robot_cell_real.xacro" /> -->
     <xacro:include filename="$(find ur5e_cell_description)/urdf/robot_cell.xacro" />
     <xacro:include filename="$(find ur_description)/urdf/ur_macro.xacro" />
+    <xacro:property name="gripper_name" value="shunk_egp50" />
+    <xacro:property name="initial_positions_file" default="$(find ur5e_cell_description)/config/initial_positions.yaml" />
     <xacro:arg name="name" default="ur5e" />
     <xacro:arg name="ur_type" default="ur5e" />
     <xacro:arg name="prefix" default="" />
-    <xacro:arg name="joint_limit_params" default="$(find ur_description)/config/$(arg ur_type)/joint_limits.yaml" />
-    <xacro:arg name="kinematics_params" default="$(find ur_description)/config/$(arg ur_type)/default_kinematics.yaml" />
-    <xacro:arg name="physical_params" default="$(find ur_description)/config/$(arg ur_type)/physical_parameters.yaml" />
-    <xacro:arg name="visual_params" default="$(find ur_description)/config/$(arg ur_type)/visual_parameters.yaml" />
+    <xacro:arg name="joint_limit_params" default="$(find ur5e_cell_description)/config/$(arg ur_type)/joint_limits.yaml" />
+    <xacro:arg name="kinematics_params" default="$(find ur5e_cell_description)/config/$(arg ur_type)/default_kinematics.yaml" />
+    <xacro:arg name="physical_params" default="$(find ur5e_cell_description)/config/$(arg ur_type)/physical_parameters.yaml" />
+    <xacro:arg name="visual_params" default="$(find ur5e_cell_description)/config/$(arg ur_type)/visual_parameters.yaml" />
     <xacro:arg name="transmission_hw_interface" default="" />
     <xacro:arg name="safety_limits" default="false" />
@@ -36,10 +37,8 @@
     <xacro:arg name="sim_ignition" default="false" />
     <xacro:arg name="simulation_controllers" default="" />
-    <xacro:arg name="initial_positions_file" default="$(find ur_description)/config/initial_positions.yaml" />
+    <xacro:arg name="initial_positions_file" default="$(find ur5e_cell_description)/config/initial_positions.yaml" />
     <xacro:arg name="use_nominal_extrinsics" default="false" />
     <xacro:arg name="add_plug" default="false" />
     <xacro:arg name="use_mesh" default="true" />
-    <xacro:property name="gripper_name" value="shunk_egp50" />
-    <xacro:property name="initial_positions_file" default="$(arg initial_positions_file)" />
     <xacro:schunk_egp50 />
     <xacro:ur_robot

File: ur5e_cell_msa_config/config/ur5e_workcell.ros2_control.xacro (robot description, xacro)
@@ -10,61 +10,43 @@
             <joint name="shoulder_pan_joint">
                 <command_interface name="position"/>
-                <command_interface name="velocity"/>
-                <command_interface name="effort"/>
                 <state_interface name="position">
                   <param name="initial_value">${initial_positions['shoulder_pan_joint']}</param>
                 </state_interface>
                 <state_interface name="velocity"/>
-                <state_interface name="effort"/>
             </joint>
             <joint name="shoulder_lift_joint">
                 <command_interface name="position"/>
-                <command_interface name="velocity"/>
-                <command_interface name="effort"/>
                 <state_interface name="position">
                   <param name="initial_value">${initial_positions['shoulder_lift_joint']}</param>
                 </state_interface>
                 <state_interface name="velocity"/>
-                <state_interface name="effort"/>
             </joint>
             <joint name="elbow_joint">
                 <command_interface name="position"/>
-                <command_interface name="velocity"/>
-                <command_interface name="effort"/>
                 <state_interface name="position">
                   <param name="initial_value">${initial_positions['elbow_joint']}</param>
                 </state_interface>
                 <state_interface name="velocity"/>
-                <state_interface name="effort"/>
             </joint>
             <joint name="wrist_1_joint">
                 <command_interface name="position"/>
-                <command_interface name="velocity"/>
-                <command_interface name="effort"/>
                 <state_interface name="position">
                   <param name="initial_value">${initial_positions['wrist_1_joint']}</param>
                 </state_interface>
                 <state_interface name="velocity"/>
-                <state_interface name="effort"/>
             </joint>
             <joint name="wrist_2_joint">
                 <command_interface name="position"/>
-                <command_interface name="velocity"/>
-                <command_interface name="effort"/>
                 <state_interface name="position">
                   <param name="initial_value">${initial_positions['wrist_2_joint']}</param>
                 </state_interface>
                 <state_interface name="velocity"/>
-                <state_interface name="effort"/>
             </joint>
             <joint name="wrist_3_joint">
                 <command_interface name="position"/>
-                <command_interface name="velocity"/>
-                <command_interface name="effort"/>
                 <state_interface name="position">
                   <param name="initial_value">${initial_positions['wrist_3_joint']}</param>
                 </state_interface>
                 <state_interface name="velocity"/>
-                <state_interface name="effort"/>
             </joint>
         </ros2_control>

Commit message: Make workcell.urdf.xacro more nice
Signed-off-by: Christoph Hellmann Santos <christoph.hellmann.santos@ipa.fraunhofer.de>

File: ur5e_cell_description/urdf/workcell.urdf.xacro (robot description, xacro)
@@ -1,10 +1,11 @@
 <?xml version="1.0"?>
 <robot xmlns:xacro="http://www.ros.org/wiki/xacro" name="ur5e_workcell">
-    <!-- loading robot  from ur5e_cell_description package-->
+    <!-- inlcuding robot cell -->
+    <xacro:include filename="$(find ur5e_cell_description)/urdf/robot_cell.xacro" />
+    <!-- inlcuding components for loading xacros -->
     <xacro:include filename="$(find ur5e_cell_description)/urdf/shunk_egp50.xacro" />
-    <xacro:include filename="$(find ur5e_cell_description)/urdf/robot_cell.xacro" />
     <xacro:include filename="$(find ur_description)/urdf/ur_macro.xacro" />
-    <xacro:property name="gripper_name" value="shunk_egp50" />
-    <xacro:property name="initial_positions_file" default="$(find ur5e_cell_description)/config/initial_positions.yaml" />
+    <xacro:include filename="$(find realsense2_description)/urdf/_d435.urdf.xacro" />
+    <!-- Args related to realsense -->
     <xacro:arg name="name" default="ur5e" />
     <xacro:arg name="ur_type" default="ur5e" />
@@ -38,8 +39,12 @@
     <xacro:arg name="simulation_controllers" default="" />
     <xacro:arg name="initial_positions_file" default="$(find ur5e_cell_description)/config/initial_positions.yaml" />
-    <xacro:arg name="use_nominal_extrinsics" default="false" />
+    <!-- Set arg initial_positions_file as property -->
+    <xacro:property name="initial_positions_file" default="$(arg initial_positions_file)" />
+    <!-- Args related to realsense -->
+    <xacro:arg name="use_nominal_extrinsics" default="false"/>
     <xacro:arg name="add_plug" default="false" />
     <xacro:arg name="use_mesh" default="true" />
-    <xacro:schunk_egp50 />
+    <!-- Robot cell is directly included from its xacro as it is no macro. -->
+    <!-- Instantiate UR robot. -->
     <xacro:ur_robot
         name="$(arg name)"
@@ -59,5 +64,5 @@
         sim_ignition="$(arg sim_ignition)"
         headless_mode="$(arg headless_mode)"
-        initial_positions="${load_yaml(initial_positions_file)}"
+        initial_positions="${xacro.load_yaml(initial_positions_file)}"
         use_tool_communication="$(arg use_tool_communication)"
         tool_voltage="$(arg tool_voltage)"
@@ -76,23 +81,34 @@
         <origin xyz="${robot_center_offset_length} ${robot_center_offset_width} ${robot_base_height}" rpy="0 0 ${pi/2}" /> <!-- position robot in the world -->
     </xacro:ur_robot>
-    <xacro:if value="$(arg sim_gazebo)">
-        <!-- Gazebo plugins -->
-        <gazebo reference="world"></gazebo>
-        <gazebo>
-            <plugin filename="libgazebo_ros2_control.so" name="gazebo_ros2_control">
-                <parameters>$(arg simulation_controllers)</parameters>
-            </plugin>
-        </gazebo>
-    </xacro:if>
+    <!-- Instantiate gripper. -->
+    <xacro:schunk_egp50 />
+    <!-- Instantiate camera. -->
+    <xacro:sensor_d435
+        parent="tool0"
+        use_nominal_extrinsics="$(arg use_nominal_extrinsics)"
+        add_plug="$(arg add_plug)"
+        use_mesh="$(arg use_mesh)"
+    >
+        <origin xyz="0 -0.05 0" rpy="${pi/2} ${pi/2} 0"/>
+    </xacro:sensor_d435>
+    <!-- Add world link -->
     <link name="world" />
-    <joint name="world_to_robot_cell_joint" type="fixed">
+    <!-- Add joint between robotcell and world -->
+    <joint
+        name="world_to_robot_cell_joint"
+        type="fixed"
+    >
         <parent link="world" />
         <child link="robotcell_base_link" />
         <origin xyz="0 0 0" rpy="0 0 0" />
     </joint>
-    <joint name="robot_to_gripper_joint" type="fixed">
+    <!-- Add joint between gripper and robot -->
+    <joint
+        name="robot_to_gripper_joint"
+        type="fixed"
+    >
         <parent link="tool0" />
-        <child link="${gripper_name}_base_link" />
-        <origin xyz="0.0 0.0 0.0" rpy="0.0 0.0 0.0" />
+        <child link="shunk_egp50_base_link" />
+        <origin xyz="0 0 0" rpy="0 0 0" />
     </joint>
 </robot>
